File: smd_esp8266.brd (EAGLE design)
At the start: 60.9 x 26.3 mm, 21 parts, among them IC1 LM1117S, IC2 DS3231/SO, U1 ESP8266-12E/ESP-12E

Commit message: grounded top and bottom planes
Parts:
- C1, C2: value (none) -> 100nF
Changed lines of the file:
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@@
 <drawing>
 <settings>
-<setting alwaysvectorfont="no"/>
+<setting alwaysvectorfont="yes"/>
 <setting verticaltext="up"/>
 </settings>
@@
 <attribute name="VALUE" x="50.03" y="-1.27" size="1.27" layer="27"/>
 </element>
-<element name="C1" library="rcl" library_urn="urn:adsk.eagle:library:334" package="C0805" package3d_urn="urn:adsk.eagle:package:23617/2" value="" x="46.99" y="17.78" smashed="yes" rot="R90">
+<element name="C1" library="rcl" library_urn="urn:adsk.eagle:library:334" package="C0805" package3d_urn="urn:adsk.eagle:package:23617/2" value="100nF" x="46.99" y="17.78" smashed="yes" rot="R90">
 <attribute name="NAME" x="45.72" y="17.78" size="1.27" layer="25" rot="R90"/>
 <attribute name="POPULARITY" value="88" x="46.99" y="17.78" size="1.778" layer="27" rot="R90" display="off"/>
@@
 <attribute name="VALUE" x="49.53" y="16.51" size="1.27" layer="27" rot="R90"/>
 </element>
-<element name="C2" library="rcl" library_urn="urn:adsk.eagle:library:334" package="C0805" package3d_urn="urn:adsk.eagle:package:23617/2" value="" x="46.99" y="12.7" smashed="yes" rot="R90">
+<element name="C2" library="rcl" library_urn="urn:adsk.eagle:library:334" package="C0805" package3d_urn="urn:adsk.eagle:package:23617/2" value="100nF" x="46.99" y="12.7" smashed="yes" rot="R90">
 <attribute name="NAME" x="44.45" y="13.97" size="1.27" layer="25" rot="R270"/>
 <attribute name="POPULARITY" value="88" x="46.99" y="12.7" size="1.778" layer="27" rot="R90" display="off"/>
